Commit message: yep

File: nodes/simple_urdf/urdf/robot (Kopie).urdf (robot description, URDF)
Before this commit: robot simple_example, 3 links, 2 joints
Joints:
- removed joint world_to_base_link=
- added joint world_to_base_joint: type fixed, parent world, child base_link, origin xyz=0.0 0.0 0.0 rpy=0.0 0.0 0.0, axis 0 0 1

File: nodes/simple_urdf/urdf/robot_alt.urdf (robot description, URDF)
Before this commit: robot simple_example, 3 links, 2 joints
Links:
- removed link world
- added link dummy
Joints:
- removed joint world_to_base_link=
- added joint dummy_joint: type fixed, parent dummy, child base_link
