Commit message: VL53

File: urdf_tb3_description/VL53L0X_changes_to_turtlebot3_package/new urdf with VL53_left and VL53_right/turtlebot3_burger.gazebo.xacro (robot description, xacro)
@@ -135,5 +135,5 @@
                 <samples>5</samples>
                 <resolution>1.0</resolution>
-                <min_angle>-0.01</min_angle>   <!-- VL53 verkleinern  was 0.25-->
+                <min_angle>-0.1</min_angle>   <!-- VL53 verkleinern  was 0.25-->
                 <max_angle>0.01</max_angle>
               </horizontal>
@@ -141,6 +141,6 @@
                 <samples>5</samples>
                 <resolution>1</resolution>
-                <min_angle>-0.01</min_angle>
-                <max_angle>0.01</max_angle>
+                <min_angle>-0.1</min_angle>
+                <max_angle>0.1</max_angle>
               </vertical>
             </scan>

File: urdf_tb3_description/VL53L0X_changes_to_turtlebot3_package/new urdf with VL53_left and VL53_right/turtlebot3_burger.urdf.xacro (robot description, xacro)
@@ -156,5 +156,5 @@
         <origin xyz="0 0 0" rpy="0 0 0"/>
         <geometry>
-            <box size="0.05 0.02 0.01"/>
+            <box size="0.005 0.02 0.01"/>
         </geometry>
         </collision>    <visual>
